File: Quests/NaOschup-2.0/NaOshupSound_2.0.kicad_pcb (KiCad board)
At the start: 2 copper layers, 102 x 86 mm, 56 parts, among them J1 Conn_01x03_Pin, J10 Conn_01x03, J11 Conn_01x03, J12 Conn_01x03, J13 Conn_01x02, J14 Conn_01x02, J15 Conn_01x02, J16 Conn_01x02, J17 Conn_01x02, J18 Conn_01x02, J19 Conn_01x02, J2 Conn_02x01, J20 Conn_01x02, J21 Conn_02x04_Odd_Even, J22 Conn_02x20_Odd_Even, J25 Conn_02x01, J26 Conn_02x01, J27 Conn_02x01, J28 Conn_01x02, J29 Conn_01x02, J3 Conn_01x02_Pin, J30 Conn_01x02, J31 Conn_01x02, J4 Conn_01x02, J5 Conn_01x02, J6 Conn_01x02, J7 AudioJack3_SwitchTR, J8 Conn_01x02, J9 Conn_01x02, Q1 IRLZ44N, Q2 IRLZ44N, Q3 IRLZ44N, U2 LM7805_TO220, U3 74AHCT125

Commit message: rfid
Parts:
- added J23: RFID1, Connector_IDC:IDC-Header_2x04_P2.54mm_Vertical, B.Cu at (36.5, 66.0)
- added J24: RFID2/SPI, Connector_IDC:IDC-Header_2x04_P2.54mm_Vertical, B.Cu at (47.5, 66.0)
- moved R5 4.06 mm to (88.0, 91.5), turned to -90 degrees
- moved R4 0.50 mm to (73.2, 88.5)
Connections:
- net /aux10 renamed RFID1_SS
- net /aux11 renamed RFID1_RST
- net /aux12 renamed RFID2_SS
- net /aux13 renamed RFID2_RST
- net Net-(A2-MOSI) renamed MOSI
- net Net-(A2-SCLK) renamed SCK
- net Net-(A3-D50_MISO) renamed MISO
- A3 pad 3V31: unconnected-(A3-3.3V-Pad3V31) -> 3V3
- A3 pad 3V32: unconnected-(A3-3.3V-Pad3V32) -> 3V3
Routing:
- net 3V3: track 0.00 -> 110.0 mm, vias 0 -> 1
- net RFID1_SS: track 73.5 -> 154.8 mm
- net RFID1_RST: track 71.5 -> 144.3 mm
- net RFID2_SS: track 73.0 -> 139.9 mm
- net RFID2_RST: track 74.3 -> 133.8 mm
- net MISO: track 69.2 -> 102.0 mm
- net MOSI: track 24.9 -> 56.3 mm, vias 1 -> 2
- net SCK: track 24.5 -> 42.4 mm
- net GND: track 31.7 -> 44.1 mm, vias 5 -> 8
- net Net-(J28-Pin_2): track 93.7 -> 104.9 mm
- net VCC: track 34.4 -> 27.4 mm
- net Net-(J31-Pin_2): track 69.7 -> 76.3 mm
- net Net-(J13-Pin_2): track 117.8 -> 123.5 mm
- net Net-(J14-Pin_2): track 121.8 -> 127.2 mm
- net Net-(J15-Pin_2): track 131.0 -> 136.1 mm
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Other:
- board text added: "MOSI MISO"
- board text added: "QUEST_ATMEGAPRO_ETH V2.1"
- board text added: "RST-D23 3V3"
- board text added: "RST-D25 3V3"
- board text added: "SS-D22 SCK"
- board text added: "SS-D24 SCK"
- board text added: "X GND"
- board text removed: "QUEST_ATMEGAPRO_ETH V2.0"
