File: Quests/NaOschup-2.0/NaOshupSound_2.0.kicad_sch (KiCad schematic)
At the start: 52 parts, among them J1 Conn_01x03_Pin, J10 Conn_01x03, J11 Conn_01x03, J12 Conn_01x03, J13 Conn_01x02, J14 Conn_01x02, J15 Conn_01x02, J16 Conn_01x02, J17 Conn_01x02, J18 Conn_01x02, J19 Conn_01x02, J2 Conn_02x01, J20 Conn_01x02, J21 Conn_02x04_Odd_Even, J22 Conn_02x20_Odd_Even, J25 Conn_02x01, J26 Conn_02x01, J27 Conn_02x01, J28 Conn_01x02, J29 Conn_01x02, J3 Conn_01x02_Pin, J30 Conn_01x02, J31 Conn_01x02, J4 Conn_01x02, J5 Conn_01x02, J6 Conn_01x02, J7 AudioJack3_SwitchTR, J8 Conn_01x02, J9 Conn_01x02, Q1 IRLZ44N, Q2 IRLZ44N, Q3 IRLZ44N, U2 LM7805_TO220, U3 74AHCT125

Commit message: rfid
Parts:
- added J23: RFID1, Connector_IDC:IDC-Header_2x04_P2.54mm_Vertical, symbol Connector_Generic:Conn_02x04_Odd_Even
- added J24: RFID2/SPI, Connector_IDC:IDC-Header_2x04_P2.54mm_Vertical, symbol Connector_Generic:Conn_02x04_Odd_Even
Connections:
- net GND: now also J23.6 (GND), J24.6 (GND)
- net 3V3: now reaches A3.3V31 (3.3V)
- net 3V3: now also A3.3V32 (3.3V), J23.8 (VCC_3V3), J24.8 (VCC_3V3)
- net MISO: now reaches A3.D50 (D50_MISO), U3.3
- net MISO: now also J23.4 (MISO), J24.4 (MISO)
- net MOSI: now reaches A2.6 (MOSI), A3.D51 (D51_MOSI)
- net MOSI: now also J23.3 (MOSI), J24.3 (MOSI)
- net SCK: now reaches A2.2 (SCLK), A3.D52 (D52_SCK)
- net SCK: now also J23.2 (SCK), J24.2 (SCK)
- net aux10 renamed RFID1_SS
- net RFID1_SS: now also J23.1 (SS)
- net aux11 renamed RFID1_RST
- net RFID1_RST: now also J23.7 (RST)
- net aux12 renamed RFID2_SS
- net RFID2_SS: now also J24.1 (SS)
- net aux13 renamed RFID2_RST
- net RFID2_RST: now also J24.7 (RST)
- no-connect marks 25 -> 23
